Commit message: Modified urdf, yaml and launch files

File: urdf/omnidirectional_four-wheeled_robot.urdf (robot description, URDF)
Before this commit: robot omnidirectional_four-wheeled_robot, 10 links, 9 joints
Links:
- removed link leftBackWheel_link1
- removed link leftBackWheel_link2
- removed link leftFrontWheel_link1
- removed link leftFrontWheel_link2
- removed link rightBackWheel_link1
- removed link rightBackWheel_link2
- removed link rightFrontWheel_link1
- removed link rightFrontWheel_link2
- added link FLwheel_link1, mass 0.500; collision cylinder length=0.1 radius=0.2; visual cylinder length=0.1 radius=0.2
- added link FLwheel_link2, mass 0.500; collision cylinder length=0.1 radius=0.2; visual cylinder length=0.1 radius=0.2
- added link FRwheel_link1, mass 2.; collision cylinder length=0.1 radius=0.2; visual cylinder length=0.1 radius=0.2
- added link FRwheel_link2, mass 2.; collision cylinder length=0.1 radius=0.2; visual cylinder length=0.1 radius=0.2
- added link RLwheel_link1, mass 0.5; collision cylinder length=0.1 radius=0.2; visual cylinder length=0.1 radius=0.2
- added link RLwheel_link2, mass 0.5; collision cylinder length=0.1 radius=0.2; visual cylinder length=0.1 radius=0.2
- added link RRwheel_link1, mass 0.500; collision cylinder length=0.1 radius=0.2; visual cylinder length=0.1 radius=0.2
- added link RRwheel_link2, mass 0.500; collision cylinder length=0.1 radius=0.2; visual cylinder length=0.1 radius=0.2
Joints:
- removed joint leftBackWheel_joint1
- removed joint leftBackWheel_joint2
- removed joint leftFrontWheel_joint1
- removed joint leftFrontWheel_joint2
- removed joint rightBackWheel_joint1
- removed joint rightBackWheel_joint2
- removed joint rightFrontWheel_joint1
- removed joint rightFrontWheel_joint2
- added joint FLwheel_joint1: type revolute, parent body_link, child FLwheel_link1, origin xyz=0.375 -0.375 0. rpy=-1.57 0. 0., axis 0. 1. 0., limit lower=-1.57 upper=1.57 effort=1. velocity=5.
- added joint FLwheel_joint2: type continuous, parent FLwheel_link1, child FLwheel_link2, origin xyz=0. 0. 0. rpy=0. 0. 0., axis 0. 0. 1.
- added joint FRwheel_joint1: type revolute, parent body_link, child FRwheel_link1, origin xyz=0.375 0.375 0. rpy=-1.57 0. 0., axis 0. 1. 0., limit lower=-1.57 upper=1.57 effort=1. velocity=5.
- added joint FRwheel_joint2: type continuous, parent FRwheel_link1, child FRwheel_link2, origin xyz=0. 0. 0. rpy=0. 0. 0., axis 0. 0. 1.
- added joint RLwheel_joint1: type revolute, parent body_link, child RLwheel_link1, origin xyz=-0.375 -0.375 0. rpy=-1.57 0. 0., axis 0. 1. 0., limit lower=-1.57 upper=1.57 effort=1. velocity=5.
- added joint RLwheel_joint2: type continuous, parent RLwheel_link1, child RLwheel_link2, origin xyz=0. 0. 0. rpy=0. 0. 0., axis 0. 0. 1.
- added joint RRwheel_joint1: type revolute, parent body_link, child RRwheel_link1, origin xyz=-0.375 0.375 0. rpy=-1.57 0. 0., axis 0. 1. 0., limit lower=-1.57 upper=1.57 effort=1. velocity=5.
- added joint RRwheel_joint2: type continuous, parent RRwheel_link1, child RRwheel_link2, origin xyz=0. 0. 0. rpy=0. 0. 0., axis 0. 0. 1.
