Commit message: 20200806 全方向移動ロボット xacroを利用したプログラムへ移行

File: urdf/omnidirectional_four-wheeled_robot.urdf.xacro (robot description, xacro)
@@ -8,13 +8,14 @@
 <!-- =================================================================================== -->
 <robot name="omnidirectional_four-wheeled_robot" xmlns:xacro="http://ros.org/wiki/xacro">
-<xacro:property name="x_side" value="0.75" />
-<xacro:property name="y_side" value="0.75" />
-<xacro:property name="z_side"  value="0.25" />
-<xacro:property name="body_mass"  value="1." />
-<xacro:property name="cylinder_radius"  value="0.2" />
-<xacro:property name="cylinder_length"  value="0.1" />
-<xacro:property name="wheel_mass" value="0.5" />
+<xacro:property name="pi" value="3.1415926535897931"/>
+<xacro:property name="x_side" value="0.75"/>
+<xacro:property name="y_side" value="0.75"/>
+<xacro:property name="z_side" value="0.25"/>
+<xacro:property name="body_mass" value="1."/>
+<xacro:property name="cylinder_radius" value="0.2"/>
+<xacro:property name="cylinder_length" value="0.1"/>
+<xacro:property name="wheel_mass" value="0.5"/>
 	<link name="base_link"/>
-	<link name="base_link">
+	<link name="body_link">
 		<visual>
 			<geometry>
@@ -33,7 +34,7 @@
 			<origin xyz="0. 0. 0."/>
 			<mass value="${body_mass}"/>
-			<inertia ixx="${body_mass * (y_side^2 + z_side^2) / 12}" ixy="0." ixz="0."
-					  iyy="${body_mass * (x_side^2 + z_side^2) / 12}" iyz="0."
-					  izz="${body_mass * (x_side^2 + y_side^2) / 12}"/>
+			<inertia ixx="${body_mass * (y_side**2 + z_side**2) / 12}" ixy="0." ixz="0."
+					  iyy="${body_mass * (x_side**2 + z_side**2) / 12}" iyz="0."
+					  izz="${body_mass * (x_side**2 + y_side**2) / 12}"/>
 		</inertial>
 	</link>
