Commit message: xacroファイル修正

File: urdf/wheel.urdf.xacro (robot description, xacro)
@@ -1,47 +1,103 @@
 <?xml version="1.0"?>
 <!-- =================================================================================== -->
-<!-- |    ommidirecctional_four-wheeled_robot.urdf.xacro							| -->
+<!-- |    wheel.urdf.xacro																| -->
 <!-- |    author: Koji Shibata                               							| -->
-<!-- |    e-mail: kshibata.0519@gmail.com											| -->
-<!-- |    This is a URDF file that describes an omnidirectional 					| -->
-<!-- |    four-wheeled robot for ROS users.											| -->
+<!-- |    e-mail: kshibata.0519@gmail.com												| -->
+<!-- |    This is a URDF file that describes an omnidirectional 						| -->
+<!-- |    four-wheeled robot for ROS users.												| -->
 <!-- =================================================================================== -->
-<robot name="omnidirectional_four-wheeled_robot" xmlns:xacro="http://ros.org/wiki/xacro">
-<xacro:property name="x_side" value="0.75" />
-<xacro:property name="y_side" value="0.75" />
-<xacro:property name="z_side"  value="0.25" />
-<xacro:property name="body_mass"  value="1." />
-<xacro:property name="cylinder_radius"  value="0.2" />
-<xacro:property name="cylinder_length"  value="0.1" />
-<xacro:property name="wheel_mass" value="0.5" />
-	<link name="base_link"/>
-	<link name="base_link">
-		<visual>
-			<geometry>
-				<box size="${x_side} ${y_side} ${z_side}"/>
-			</geometry>
-			<material name="White">
-				<color rgba="1. 1. 1. 1."/>
-			</material>
-		</visual>
-		<collision>
-			<geometry>
-				<box size="${x_side} ${y_side} ${z_side}"/>
-			</geometry>
-		</collision>
-		<inertial>
-			<origin xyz="0. 0. 0."/>
-			<mass value="${body_mass}"/>
-			<inertia ixx="${body_mass * (y_side^2 + z_side^2) / 12}" ixy="0." ixz="0."
-					  iyy="${body_mass * (x_side^2 + z_side^2) / 12}" iyz="0."
-					  izz="${body_mass * (x_side^2 + y_side^2) / 12}"/>
-		</inertial>
-	</link>
-	<joint name="base_joint" type="fixed">
-		<origin xyz="0. 0. 0.3" rpy="0. 0. 0."/>
-		<parent link="base_link"/>
-		<child link="body_link"/>
-		<calibration rising="0."/>
-		<dynamics damping="0." friction="0."/>
-	 </joint>
+<robot xmlns:xacro="http://ros.org/wiki/xacro">
+	<xacro:macro name="wheel_macro" params="suffix parent x_pos y_pos">
+		<link name="${suffix}_link1">
+			<visual>
+				<geometry>
+					<cylinder radius="${cylinder_radius}" length="${cylinder_length}"/>
+				</geometry>
+				<material name="Black">
+					<color rgba="0. 0. 0. 1."/>
+				</material>
+			</visual>
+			<collision>
+				<geometry>
+					<cylinder radius="${cylinder_radius}" length="${cylinder_length}"/>
+				</geometry>
+			</collision>
+			<inertial>
+				<origin xyz="0. 0. 0."/>
+				<mass value="${wheel_mass}"/>
+				<inertia ixx="${wheel_mass * cylinder_radius**2 / 2}" ixy="0." ixz="0."
+						 iyy="${wheel_mass * (cylinder_radius**2 / 4 + cylinder_length**2 / 12)}" iyz="0."
+						 izz="${wheel_mass * (cylinder_radius**2 / 4 + cylinder_length**2 / 12)}"/>
+			</inertial>
+		</link>
+		<link name="${suffix}_link2">
+			<visual>
+				<geometry>
+					<cylinder radius="${cylinder_radius}" length="${cylinder_length}"/>
+				</geometry>
+				<material name="Black">
+					<color rgba="0. 0. 0. 1."/>
+				</material>
+			</visual>
+			<collision>
+				<geometry>
+					<cylinder radius="${cylinder_radius}" length="${cylinder_length}"/>
+				</geometry>
+			</collision>
+			<inertial>
+				<origin xyz="0. 0. 0."/>
+				<mass value="${wheel_mass}"/>
+				<inertia ixx="${wheel_mass * cylinder_radius**2 / 2}" ixy="0." ixz="0."
+						 iyy="${wheel_mass * (cylinder_radius**2 / 4 + cylinder_length**2 / 12)}" iyz="0."
+						 izz="${wheel_mass * (cylinder_radius**2 / 4 + cylinder_length**2 / 12)}"/>
+			</inertial>
+		</link>
+		<joint name="${suffix}_joint1" type="revolute">
+			<limit lower="-${pi/2}" upper="${pi/2}" effort="${effort_limit}" velocity="${velocity_limit}"/>
+			<origin xyz="${x_pos} ${y_pos} 0." rpy="-${pi/2} 0. 0."/>
+			<axis xyz="0. 1. 0."/>
+			<parent link="${parent}"/>
+			<child link="${suffix}_link1"/>
+			<calibration rising="0."/>
+			<dynamics damping="0." friction="0."/>
+		</joint>
+		<joint name="${suffix}_joint2" type="continuous">
+			<origin xyz="0. 0. 0." rpy="0. 0. 0."/>
+			<axis xyz="0. 0. 1."/>
+			<parent link="${suffix}_link1"/>
+			<child link="${suffix}_link2"/>
+			<calibration rising="0."/>
+			<dynamics damping="0." friction="0."/>
+		</joint>
+		<transmission name="${suffix}_trans1">
+			<type>transmission_interface/SimpleTransmission</type>
+			<joint name="${suffix}_joint1">
+				<hardwareInterface>hardware_interface/PositionJointInterface</hardwareInterface>
+			</joint>
+			<actuator name="${suffix}_motor1">
+				<mechanicalReduction>1</mechanicalReduction>
+				<hardwareInterface>hardware_interface/PositionJointInterface</hardwareInterface>
+			</actuator>
+		</transmission>
+		<transmission name="${suffix}_trans2">
+			<type>transmission_interface/SimpleTransmission</type>
+			<joint name="${suffix}_joint2">
+				<hardwareInterface>hardware_interface/VelocityJointInterface</hardwareInterface>
+			</joint>
+			<actuator name="${suffix}_motor2">
+				<mechanicalReduction>1</mechanicalReduction>
+				<hardwareInterface>hardware_interface/VelocityJointInterface</hardwareInterface>
+			</actuator>
+		</transmission>
+		<gazebo reference="${suffix}_link1">
+			<selfCollide>false</selfCollide>
+			<mu1 value="0.05"/>
+			<mu2 value="0.05"/>
+		</gazebo>
+		<gazebo reference="${suffix}_link2">
+			<selfCollide>false</selfCollide>
+			<mu1 value="0.80"/>
+			<mu2 value="0.80"/>
+		</gazebo>
+	</xacro:macro>
 </robot>
