Commit message: xacroファイル修正

File: urdf/camera.urdf.xacro (robot description, xacro)
@@ -1,10 +1,10 @@
 <?xml version="1.0"?>
-<!-- =================================================================================== -->
-<!-- |    camera.urdf.xacro																| -->
-<!-- |    author: Koji Shibata															| -->
-<!-- |    e-mail: kshibata.0519@gmail.com　												| -->
-<!-- |    This is a URDF file that describes an omnidirectional 						| -->
-<!-- |    four-wheeled robot for ROS users. 											| -->
-<!-- =================================================================================== -->
+<!-- ===========================================================================  -->
+<!-- |    camera.urdf.xacro																											| -->
+<!-- |    author: Koji Shibata                               										| -->
+<!-- |    e-mail: kshibata.0519@gmail.com																				| -->
+<!-- |    This is a URDF file that describes an omnidirectional 								| -->
+<!-- |    four-wheeled robot for ROS users.																			| -->
+<!-- ===========================================================================  -->
 <robot xmlns:xacro="http://ros.org/wiki/xacro">
   <xacro:macro name="camera_macro" params="parent prefix xyz">

File: urdf/laser.urdf.xacro (robot description, xacro)
@@ -1,10 +1,10 @@
 <?xml version="1.0"?>
-<!-- =================================================================================== -->
-<!-- |    laser.urdf.xacro															| -->
-<!-- |    author: Koji Shibata														| -->
-<!-- |    e-mail: kshibata.0519@gmail.com　											| -->
-<!-- |    This is a URDF file that describes an omnidirectional 					| -->
-<!-- |    four-wheeled robot for ROS users. 										| -->
-<!-- =================================================================================== -->
+<!-- ===========================================================================  -->
+<!-- |    laser.urdf.xacro																											| -->
+<!-- |    author: Koji Shibata                               										| -->
+<!-- |    e-mail: kshibata.0519@gmail.com																				| -->
+<!-- |    This is a URDF file that describes an omnidirectional 								| -->
+<!-- |    four-wheeled robot for ROS users.																			| -->
+<!-- ===========================================================================  -->
 <robot xmlns:xacro="http://ros.org/wiki/xacro">
 	<xacro:macro name="laser_macro" params="parent prefix xyz rpy">

File: urdf/robot.urdf.xacro (robot description, xacro)
@@ -1,14 +1,14 @@
 <?xml version="1.0"?>
-<!-- ==================================================================================== -->
-<!-- |    ommidirecctional_four-wheeled_robot.urdf.xacro								| -->
-<!-- |    author: Koji Shibata                               							| -->
-<!-- |    e-mail: kshibata.0519@gmail.com												| -->
-<!-- |    This is a URDF file that describes an omnidirectional 						| -->
-<!-- |    four-wheeled robot for ROS users.												| -->
-<!-- ==================================================================================== -->
+<!-- ===========================================================================  -->
+<!-- |    ommidirecctional_four-wheeled_robot.urdf.xacro												| -->
+<!-- |    author: Koji Shibata                               										| -->
+<!-- |    e-mail: kshibata.0519@gmail.com																				| -->
+<!-- |    This is a URDF file that describes an omnidirectional 								| -->
+<!-- |    four-wheeled robot for ROS users.																			| -->
+<!-- ===========================================================================  -->
 <robot name="omnidirectional_four-wheeled_robot" xmlns:xacro="http://ros.org/wiki/xacro">
-<xacro:property name="x_side" value="0.75"/>
-<xacro:property name="y_side" value="0.75"/>
-<xacro:property name="z_side" value="0.25"/>
+<xacro:property name="x_size" value="0.75"/>
+<xacro:property name="y_size" value="0.75"/>
+<xacro:property name="z_size" value="0.25"/>
 <xacro:property name="body_mass" value="1."/>
 <xacro:property name="cylinder_radius" value="0.2"/>
@@ -25,5 +25,5 @@
 		<visual>
 			<geometry>
-				<box size="${x_side} ${y_side} ${z_side}"/>
+				<box size="${x_size} ${y_size} ${z_size}"/>
 			</geometry>
 			<material name="White">
@@ -33,5 +33,5 @@
 		<collision>
 			<geometry>
-				<box size="${x_side} ${y_side} ${z_side}"/>
+				<box size="${x_size} ${y_size} ${z_size}"/>
 			</geometry>
 		</collision>
@@ -39,7 +39,27 @@
 			<origin xyz="0. 0. 0."/>
 			<mass value="${body_mass}"/>
-			<inertia ixx="${body_mass * (y_side**2 + z_side**2) / 12}" ixy="0." ixz="0."
-					 iyy="${body_mass * (x_side**2 + z_side**2) / 12}" iyz="0."
-					 izz="${body_mass * (x_side**2 + y_side**2) / 12}"/>
+			<inertia ixx="${body_mass * (y_size**2 + z_size**2) / 12}" ixy="0." ixz="0."
+					  iyy="${body_mass * (x_size**2 + z_size**2) / 12}" iyz="0."
+					  izz="${body_mass * (x_size**2 + y_size**2) / 12}"/>
+		</inertial>
+	</link>
+	<link name="frontPoint_link">
+		<visual>
+			<geometry>
+				<box size="0.05 0.05 0.05"/>
+			</geometry>
+			<material name="Red">
+				<color rgba="1. 0. 0. 1."/>
+			</material>
+		</visual>
+		<collision>
+			<geometry>
+				<box size="0.05 0.05 0.05"/>
+			</geometry>
+		</collision>
+		<inertial>
+			<origin xyz="0. 0. 0."/>
+			<mass value="0."/>
+			<inertia ixx="0." ixy="0." ixz="0." iyy="0." iyz="0." izz="0."/>
 		</inertial>
 	</link>
@@ -51,15 +71,24 @@
 		<dynamics damping="0." friction="0."/>
 	</joint>
+	<joint name="frontPoint_joint" type="fixed">
+		<origin xyz="${x_size/2 - 0.02} 0. ${z_size/2 - 0.02}" rpy="0. 0. 0."/>
+		<parent link="body_link"/>
+		<child link="frontPoint_link"/>
+	</joint>
 	<xacro:wheel_macro suffix="FRwheel" parent="body_link" x_pos="0.375"  y_pos="0.375"/>
 	<xacro:wheel_macro suffix="RRwheel" parent="body_link" x_pos="0.375"  y_pos="-0.375"/>
 	<xacro:wheel_macro suffix="FLwheel" parent="body_link" x_pos="-0.375" y_pos="0.375"/>
 	<xacro:wheel_macro suffix="RLwheel" parent="body_link" x_pos="-0.375" y_pos="-0.375"/>
-	<xacro:camera_macro prefix="camera" parent="body_link" xyz="${x_side/2} 0. ${z_side/2}"/>
-	<xacro:laser_macro prefix="FrontLaser" parent="body_link" xyz="${x_side/4} 0. ${z_side/2 + 1.e-2}" rpy="0. 0. 0."/>
-	<xacro:laser_macro prefix="RearLaser" parent="body_link" xyz="${-x_side/4} 0. ${z_side/2 + 1.e-2}" rpy="0. 0. ${-pi}"/>
+	<xacro:camera_macro prefix="camera" parent="body_link" xyz="${x_size/2} 0. ${z_size/2}"/>
+	<!-- <xacro:laser_macro prefix="FrontLaser" parent="body_link" xyz="${x_size/4} 0. ${z_size/2 + 1.e-2}" rpy="0. 0. 0."/>
+	<xacro:laser_macro prefix="RearLaser" parent="body_link" xyz="${-x_size/4} 0. ${z_size/2 + 1.e-2}" rpy="0. 0. ${-pi}"/> -->
 	<gazebo reference="base_link">
 		<selfCollide>false</selfCollide>
 		<mu1 value="0.05"/>
 		<mu2 value="0.05"/>
+	</gazebo>
+	<gazebo reference="frontPoint_link">
+		<selfCollide>false</selfCollide>
+		<material>Gazebo/Red</material>
 	</gazebo>
 	<gazebo>

File: urdf/wheel.urdf.xacro (robot description, xacro)
@@ -1,14 +1,15 @@
 <?xml version="1.0"?>
-<!-- =================================================================================== -->
-<!-- |    wheel.urdf.xacro																| -->
-<!-- |    author: Koji Shibata                               							| -->
-<!-- |    e-mail: kshibata.0519@gmail.com												| -->
-<!-- |    This is a URDF file that describes an omnidirectional 						| -->
-<!-- |    four-wheeled robot for ROS users.												| -->
-<!-- =================================================================================== -->
+<!-- ===========================================================================  -->
+<!-- |    wheel.urdf.xacro																											| -->
+<!-- |    author: Koji Shibata                               										| -->
+<!-- |    e-mail: kshibata.0519@gmail.com																				| -->
+<!-- |    This is a URDF file that describes an omnidirectional 								| -->
+<!-- |    four-wheeled robot for ROS users.																			| -->
+<!-- ===========================================================================  -->
 <robot xmlns:xacro="http://ros.org/wiki/xacro">
 	<xacro:macro name="wheel_macro" params="suffix parent x_pos y_pos">
 		<link name="${suffix}_link1">
 			<visual>
+				<origin xyz="0. 0. 0." rpy="-${pi/2} 0. 0."/>
 				<geometry>
 					<cylinder radius="${cylinder_radius}" length="${cylinder_length}"/>
@@ -19,4 +20,5 @@
 			</visual>
 			<collision>
+				<origin xyz="0. 0. 0." rpy="-${pi/2} 0. 0."/>
 				<geometry>
 					<cylinder radius="${cylinder_radius}" length="${cylinder_length}"/>
@@ -24,13 +26,14 @@
 			</collision>
 			<inertial>
-				<origin xyz="0. 0. 0."/>
+				<origin xyz="0. 0. 0." rpy="-${pi/2} 0. 0."/>
 				<mass value="${wheel_mass}"/>
 				<inertia ixx="${wheel_mass * cylinder_radius**2 / 2}" ixy="0." ixz="0."
-						 iyy="${wheel_mass * (cylinder_radius**2 / 4 + cylinder_length**2 / 12)}" iyz="0."
-						 izz="${wheel_mass * (cylinder_radius**2 / 4 + cylinder_length**2 / 12)}"/>
+						  	 iyy="${wheel_mass * (cylinder_radius**2 / 4 + cylinder_length**2 / 12)}" iyz="0."
+						 	 	 izz="${wheel_mass * (cylinder_radius**2 / 4 + cylinder_length**2 / 12)}"/>
 			</inertial>
 		</link>
 		<link name="${suffix}_link2">
 			<visual>
+				<origin xyz="0. 0. 0." rpy="-${pi/2} 0. 0."/>
 				<geometry>
 					<cylinder radius="${cylinder_radius}" length="${cylinder_length}"/>
@@ -41,4 +44,5 @@
 			</visual>
 			<collision>
+				<origin xyz="0. 0. 0." rpy="-${pi/2} 0. 0."/>
 				<geometry>
 					<cylinder radius="${cylinder_radius}" length="${cylinder_length}"/>
@@ -46,27 +50,26 @@
 			</collision>
 			<inertial>
-				<origin xyz="0. 0. 0."/>
+				<origin xyz="0. 0. 0." rpy="-${pi/2} 0. 0."/>
 				<mass value="${wheel_mass}"/>
 				<inertia ixx="${wheel_mass * cylinder_radius**2 / 2}" ixy="0." ixz="0."
-						 iyy="${wheel_mass * (cylinder_radius**2 / 4 + cylinder_length**2 / 12)}" iyz="0."
-						 izz="${wheel_mass * (cylinder_radius**2 / 4 + cylinder_length**2 / 12)}"/>
+					  		 iyy="${wheel_mass * (cylinder_radius**2 / 4 + cylinder_length**2 / 12)}" iyz="0."
+						  	 izz="${wheel_mass * (cylinder_radius**2 / 4 + cylinder_length**2 / 12)}"/>
 			</inertial>
 		</link>
-		<joint name="${suffix}_joint1" type="revolute">
-			<limit lower="-${pi/2}" upper="${pi/2}" effort="${effort_limit}" velocity="${velocity_limit}"/>
-			<origin xyz="${x_pos} ${y_pos} 0." rpy="-${pi/2} 0. 0."/>
-			<axis xyz="0. 1. 0."/>
+		<joint name="${suffix}_joint1" type="continuous">
+			<origin xyz="${x_pos} ${y_pos} 0." rpy="0. 0. 0."/>
+			<axis xyz="0. 0. 1."/>
 			<parent link="${parent}"/>
 			<child link="${suffix}_link1"/>
 			<calibration rising="0."/>
-			<dynamics damping="0." friction="0."/>
+			<dynamics damping="1." friction="0."/>
 		</joint>
 		<joint name="${suffix}_joint2" type="continuous">
 			<origin xyz="0. 0. 0." rpy="0. 0. 0."/>
-			<axis xyz="0. 0. 1."/>
+			<axis xyz="0. 1. 0."/>
 			<parent link="${suffix}_link1"/>
 			<child link="${suffix}_link2"/>
 			<calibration rising="0."/>
-			<dynamics damping="0." friction="0."/>
+			<dynamics damping="1." friction="0."/>
 		</joint>
 		<transmission name="${suffix}_trans1">
@@ -94,4 +97,5 @@
 			<mu1 value="0.05"/>
 			<mu2 value="0.05"/>
+			<material>Gazebo/Black</material>
 		</gazebo>
 		<gazebo reference="${suffix}_link2">
@@ -99,4 +103,5 @@
 			<mu1 value="0.80"/>
 			<mu2 value="0.80"/>
+			<material>Gazebo/Black</material>
 		</gazebo>
 	</xacro:macro>
